File: motorcon/motorcon.sch (KiCad schematic (older format))
At the start: 123 parts, among them J1 Main_Batt_Con, J2 Batt_Balancer_Con, J3 Charger_Con, J4 Left_Motor, J5 Right_Motor, J6 Brush_Motor, J7 Side_Brush, J8 Conn_01x06, Q1 FCX491, Q2 CSD87312Q3E, Q3 CSD25402Q3A, Q4 CSD17307Q5A, Q5 CSD17307Q5A, U1 STM32F103C8Tx, U2 TLV73333PDBV, U3 LTC6810IG-2#3ZZPBF, U4 BQ24715RGRR, U5 TPS5450DDA, U6 DRV8876PWPR, U7 DRV8876PWPR, U8 DRV8876PWPR, U9 DRV8876PWPR

Commit message: Finished Schematic, added custom footprints
Parts:
- removed C22: 220uF, symbol Device:C
- removed D3: D, symbol Device:D
- added C43, C44: 20pF, Capacitor_SMD:C_0805_2012Metric, symbol Device:C
- added C45, C47, C48, C49, C50: 100nF, Capacitor_SMD:C_0805_2012Metric, symbol Device:C
- added C46, C51: 1uF, Capacitor_SMD:C_0805_2012Metric, symbol Device:C
- added D3: BAT54, Diode_SMD:D_SOT-23_ANK, symbol Device:D_Schottky
- added D4: LED, LED_SMD:LED_0603_1608Metric, symbol Device:LED
- added J10: SWD, Connector_PinHeader_2.54mm:PinHeader_1x03_P2.54mm_Horizontal, symbol Connector_Generic:Conn_01x03
- added J9: SPI_PI, Connector_JST:JST_PH_S4B-PH-SM4-TB_1x04-1MP_P2.00mm_Horizontal, symbol Connector_Generic:Conn_01x04
- added R55: 180, Resistor_SMD:R_0805_2012Metric, symbol Device:R
- added R56, R57, R58: 600, Resistor_SMD:R_0805_2012Metric, symbol Device:R
- added R59, R60, R61, R62: 10k, Resistor_SMD:R_0805_2012Metric, symbol Device:R
- added Y1: 8M, Crystal:Crystal_SMD_3225-4Pin_3.2x2.5mm, symbol Device:Crystal
- C1, C10, C11, C12, C13, C14, C15, C16, C17, C18, C19, C2, C20, C21, C23, C28, C29, C3, C30, C31, C32, C33, C34, C35, C36, C37, C38, C39, C4, C41, C5, C6, C8, C9: footprint (none) -> Capacitor_SMD:C_0805_2012Metric
- C24, C25, C26, C27: footprint (none) -> Capacitor_THT:C_Radial_D6.3mm_H11.0mm_P2.50mm
- C40: value 56uF -> 82uF; footprint (none) -> Capacitor_SMD:C_Elec_10x10.2
- C42: footprint (none) -> Capacitor_SMD:C_Elec_10x10.2
- C7: footprint (none) -> Capacitor_SMD:C_Elec_4x5.4
- D1, D2: footprint (none) -> Diode_SMD:D_SOT-23_ANK
- J4, J5, J6: footprint (none) -> Connector_JST:JST_PH_S5B-PH-SM4-TB_1x05-1MP_P2.00mm_Horizontal
- J7: footprint Connector_AMASS:AMASS_XT30PW-M_1x02_P2.50mm_Horizontal -> Connector_JST:JST_PH_S2B-PH-SM4-TB_1x02-1MP_P2.00mm_Horizontal
- J8: footprint (none) -> Connector_JST:JST_PH_S6B-PH-SM4-TB_1x06-1MP_P2.00mm_Horizontal
- L1: footprint (none) -> HCM1104-3R3:HCM1104-3R3
- L2: footprint (none) -> BCIHP1770HC:BCIHP1770HC
- Q1: footprint (none) -> Package_TO_SOT_SMD:SOT-89-3
- Q2: footprint DPB8 -> Resistor_SMD:R_0805_2012Metric; symbol CSD87312Q3E:CSD87312Q3E -> motorcon-rescue:CSD87312Q3E-CSD87312Q3E
- Q3: footprint CSD25402Q3A -> Resistor_SMD:R_0805_2012Metric; symbol CSD25402Q3A:CSD25402Q3A -> motorcon-rescue:CSD25402Q3A-CSD25402Q3A
- Q4, Q5: footprint DQJ8 -> Resistor_SMD:R_0805_2012Metric; symbol CSD17307Q5A:CSD17307Q5A -> motorcon-rescue:CSD17307Q5A-CSD17307Q5A
- R1, R10, R11, R12, R13, R14, R15, R16, R17, R18, R19, R2, R20, R21, R22, R23, R24, R25, R26, R27, R28, R29, R3, R30, R31, R32, R33, R34, R35, R36, R37, R38, R39, R4, R40, R41, R42, R43, R44, R45, R46, R47, R48, R49, R5, R50, R51, R52, R53, R54, R6, R7, R8, R9: footprint (none) -> Resistor_SMD:R_0805_2012Metric
- U3: footprint (none) -> LTC6810:SSOP-44; symbol LTC6810-2:LTC6810IG-2#3ZZPBF -> motorcon-rescue:LTC6810IG-2#3ZZPBF-LTC6810-2
- U4: footprint RGR20_2P05X2P05_TEX -> BQ24715RGRR:BQ24715RGRR; symbol BQ24715RGRR:BQ24715RGRR -> motorcon-rescue:BQ24715RGRR-BQ24715RGRR
- U5: footprint DDA8_3P1X2P4 -> TPS5450DDA:TPS5450DDA; symbol TPS5450DDA:TPS5450DDA -> motorcon-rescue:TPS5450DDA-TPS5450DDA
- U6, U7, U8, U9: footprint PWP0016J_N -> DRV8876PWPR:DRV8876PWPR; symbol DRV8876PWPR:DRV8876PWPR -> motorcon-rescue:DRV8876PWPR-DRV8876PWPR
Connections:
- net labels added: EncoBrush, EncoLeft, EncoRight, PC13, PD0, PD1
- wire segments 533 -> 672
Other:
- note added: "Microcontroller"
- note removed: "Needs Footprint"
- note removed: "PULL UPS"
- moved on the sheet: J4, J5, J6, J7, R35, R36, R37, R38, R39, R40, R41, R42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

Commit message: did the BOM
Parts:
- added J11: Main_Power, Connector_Molex:Molex_Mini-Fit_Jr_5569-04A2_2x02_P4.20mm_Horizontal, symbol Connector_Generic:Conn_01x04
- C1, C2, C3, C41: LCSC (none) -> C52278
- C10, C12, C13, C14, C17, C23, C4, C46, C5, C51, C6: LCSC (none) -> C282736
- C11, C15, C16, C28, C29, C30, C31, C32, C33, C34, C35, C8: LCSC (none) -> C476766
- C18, C19, C20, C21: LCSC (none) -> C17024
- C36, C37, C38, C39: LCSC (none) -> C24658
- C40: footprint Capacitor_SMD:C_Elec_10x10.2 -> Capacitor_SMD:CP_Elec_10x10; LCSC (none) -> C413517
- C42: footprint Capacitor_SMD:C_Elec_10x10.2 -> Capacitor_SMD:CP_Elec_10x10; LCSC (none) -> C359223
- C43, C44: LCSC (none) -> C94472
- C45, C47, C48, C49, C50: LCSC (none) -> C1711
- C7: LCSC (none) -> C3348
- C9: LCSC (none) -> C1790
- D1, D2: LCSC (none) -> C369922
- D3: footprint Diode_SMD:D_SOT-23_ANK -> Diode_SMD:D_SMB; LCSC (none) -> C32513
- D4: LCSC (none) -> C84263
- J1: LCSC (none) -> C431092
- J3: footprint Connector_AMASS:AMASS_XT30PW-M_1x02_P2.50mm_Horizontal -> Connector_JST:JST_VH_B2P-VH_1x02_P3.96mm_Vertical; LCSC (none) -> C138453
- L1: LCSC (none) -> C427317
- L2: value 10H -> 10uH; LCSC (none) -> C237980
- Q1: LCSC (none) -> C156315
- Q2: footprint Resistor_SMD:R_0805_2012Metric -> CSD87312Q3E:CSD87312Q3E; LCSC (none) -> C553144
- Q3: footprint Resistor_SMD:R_0805_2012Metric -> CSD25402Q3A:CSD25402Q3A; LCSC (none) -> C111356
- Q4, Q5: footprint Resistor_SMD:R_0805_2012Metric -> CSD17307Q5A:CSD17307Q5A; LCSC (none) -> C139362
- R1, R2, R3: LCSC (none) -> C334920
- R12, R13, R15, R16, R17, R18, R36, R38, R40, R42, R43, R44, R45, R46, R47, R48, R49, R50, R53, R54, R8, R9: LCSC (none) -> C17477
- R14, R23: LCSC (none) -> C149504
- R19: LCSC (none) -> C17692
- R20: LCSC (none) -> C17791
- R21, R22: LCSC (none) -> C17663
- R24, R28: footprint Resistor_SMD:R_0805_2012Metric -> Resistor_SMD:R_1206_3216Metric; LCSC (none) -> C309628
- R25, R26: LCSC (none) -> C17415
- R27, R31, R32, R33, R34, R51, R59, R60, R61, R62: LCSC (none) -> C17414
- R35, R37, R39, R41: LCSC (none) -> C170940
- R4, R5, R6: LCSC (none) -> C103902
- R52: LCSC (none) -> C17609
- R55: LCSC (none) -> C104048
- R56, R57, R58: LCSC (none) -> C17777
- R7: LCSC (none) -> C103909
- U1: LCSC (none) -> C8734
- U2: LCSC (none) -> C134139
- U4: LCSC (none) -> C276341
- U5: LCSC (none) -> C114425
- Y1: LCSC (none) -> C400090
Connections:
- net +3V3: now also R55.1
- net +5V: now also J11.1 (Pin_1)
- net GND: now also J11.3 (Pin_3), J11.4 (Pin_4); no longer R55.2
- net VCC: now also J11.2 (Pin_2)
- net at D4.1 (K): now also R55.2; no longer R55.1
Other:
- moved on the sheet: D4, R55
