File: motorcon/motorcon.sch (KiCad schematic (older format))
At the start: 144 parts, among them J1 Main_Batt_Con, J10 SWD, J11 Main_Power, J2 Batt_Balancer_Con, J3 Charger_Con, J4 Left_Motor, J5 Right_Motor, J6 Brush_Motor, J7 Side_Brush, J8 Conn_01x06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

Commit message: stuff
Parts:
- J1: footprint Connector_AMASS:AMASS_XT30PW-M_1x02_P2.50mm_Horizontal -> Connector_AMASS:AMASS_XT30U-M_1x02_P5.0mm_Vertical
- J2: footprint Connector_JST:JST_PH_S4B-PH-K_1x04_P2.00mm_Horizontal -> Connector_JST:JST_PH_B4B-PH-K_1x04_P2.00mm_Vertical
Changed lines of the file:
@@
 F 0 "J1" H 8900 1250 50  0000 C CNN
 F 1 "Main_Batt_Con" H 8950 1350 50  0000 C CNN
-F 2 "Connector_AMASS:AMASS_XT30PW-M_1x02_P2.50mm_Horizontal" H 8750 1250 50  0001 C CNN
+F 2 "Connector_AMASS:AMASS_XT30U-M_1x02_P5.0mm_Vertical" H 8750 1250 50  0001 C CNN
 F 3 "~" H 8750 1250 50  0001 C CNN
 F 4 "C431092" H 8750 1250 50  0001 C CNN "LCSC"
@@
 F 0 "J2" H 8900 1800 50  0000 C CNN
 F 1 "Batt_Balancer_Con" H 9050 1900 50  0000 C CNN
-F 2 "Connector_JST:JST_PH_S4B-PH-K_1x04_P2.00mm_Horizontal" H 8750 1700 50  0001 C CNN
+F 2 "Connector_JST:JST_PH_B4B-PH-K_1x04_P2.00mm_Vertical" H 8750 1700 50  0001 C CNN
 F 3 "~" H 8750 1700 50  0001 C CNN
 	1    8750 1700

Commit message: add
Parts:
- added J?: Conn_01x04, symbol Connector_Generic:Conn_01x04
- added Q? (x2): VBE1303, Package_TO_SOT_SMD:TO-252-2, symbol Transistor_FET:2N7000
- added R?: 1M, Resistor_SMD:R_0805_2012Metric, symbol Device:R
- J1: footprint Connector_AMASS:AMASS_XT30U-M_1x02_P5.0mm_Vertical -> Connector_AMASS:AMASS_XT30UPB-M_1x02_P5.0mm_Vertical; LCSC C431092 -> C428721
- J10: footprint Connector_PinHeader_2.54mm:PinHeader_1x03_P2.54mm_Horizontal -> Connector_JST:JST_PH_B4B-PH-K_1x04_P2.00mm_Vertical; symbol Connector_Generic:Conn_01x03 -> Connector_Generic:Conn_01x04
- J4, J5, J6: footprint Connector_JST:JST_PH_S5B-PH-SM4-TB_1x05-1MP_P2.00mm_Horizontal -> Connector_JST:JST_PH_B5B-PH-K_1x05_P2.00mm_Vertical
- J7: footprint Connector_JST:JST_PH_S2B-PH-SM4-TB_1x02-1MP_P2.00mm_Horizontal -> Connector_JST:JST_PH_B5B-PH-K_1x05_P2.00mm_Vertical
- J8: footprint Connector_JST:JST_PH_S6B-PH-SM4-TB_1x06-1MP_P2.00mm_Horizontal -> Connector_JST:JST_PH_B5B-PH-K_1x05_P2.00mm_Vertical
- J9: footprint Connector_JST:JST_PH_S4B-PH-SM4-TB_1x04-1MP_P2.00mm_Horizontal -> Connector_JST:JST_PH_B5B-PH-K_1x05_P2.00mm_Vertical
Connections:
- net labels added: Switch
- wire segments 680 -> 687
Other:
- note removed: "Main Switch"
- moved on the sheet: C43, C44, C45, C46, C47, C48, C49, C50, C51, D4, J11, J9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

Commit message: stuffs
Parts:
- removed J?: Conn_01x04, symbol Connector_Generic:Conn_01x04
- removed Q? (x2): VBE1303, Package_TO_SOT_SMD:TO-252-2, symbol Transistor_FET:2N7000
- added R?: 10k, Resistor_SMD:R_0805_2012Metric, symbol Device:R
- added SW?: SW_DIP_x01, symbol Switch:SW_DIP_x01
- gave numbers to parts that had none: 1
Connections:
- wire segments 687 -> 690
Changed lines of the file:
@@
 	7750 10450 7000 10450
 $Comp
-L power:+3.3V #PWR?
+L power:+3.3V #PWR0116
 U 1 1 5F5A19EA
 P 7650 10150
-F 0 "#PWR?" H 7650 10000 50  0001 C CNN
+F 0 "#PWR0116" H 7650 10000 50  0001 C CNN
 F 1 "+3.3V" H 7665 10323 50  0000 C CNN
 F 2 "" H 7650 10150 50  0001 C CNN
@@
 	8500 8550 8650 8550
 $Comp
-L Device:R R?
+L Device:R R63
 U 1 1 5FC05E47
 P 8650 8350
-F 0 "R?" H 8600 8450 50  0000 R CNN
+F 0 "R63" H 8600 8450 50  0000 R CNN
 F 1 "1M" H 8600 8350 50  0000 R CNN
 F 2 "Resistor_SMD:R_0805_2012Metric" V 8580 8350 50  0001 C CNN
@@
 Wire Notes Line style solid rgb(132, 0, 0)
 	500  11200 11800 11200
-$Comp
-L Transistor_FET:2N7000 Q?
-U 1 1 6004202F
-P 14650 4850
-F 0 "Q?" H 14855 4896 50  0000 L CNN
-F 1 "VBE1303" H 14855 4805 50  0000 L CNN
-F 2 "Package_TO_SOT_SMD:TO-252-2" H 14850 4775 50  0001 L CIN
-F 3 "" H 14650 4850 50  0001 L CNN
-	1    14650 4850
-	-1   0    0    -1
-$EndComp
-$Comp
-L Connector_Generic:Conn_01x04 J?
-U 1 1 60077EC3
-P 3550 9250
-F 0 "J?" H 3630 9242 50  0000 L CNN
-F 1 "Conn_01x04" H 3630 9151 50  0000 L CNN
-F 2 "" H 3550 9250 50  0001 C CNN
-F 3 "~" H 3550 9250 50  0001 C CNN
-	1    3550 9250
-	1    0    0    -1
-$EndComp
 Wire Wire Line
 	14450 5700 14550 5700
@@
 Wire Wire Line
 	14550 4650 14550 4350
-Text GLabel 14850 4850 2    50   Input ~ 0
+Text GLabel 15050 4850 2    50   Input ~ 0
 Switch
 $Comp
-L Transistor_FET:2N7000 Q?
-U 1 1 6136C1F1
-P 2650 9350
-F 0 "Q?" V 2992 9350 50  0000 C CNN
-F 1 "VBE1303" V 2901 9350 50  0000 C CNN
-F 2 "Package_TO_SOT_SMD:TO-252-2" H 2850 9275 50  0001 L CIN
-F 3 "" H 2650 9350 50  0001 L CNN
-	1    2650 9350
-	0    1    -1   0
+L Switch:SW_DIP_x01 SW?
+U 1 1 5F46B8F6
+P 1700 8100
+F 0 "SW?" H 1700 8367 50  0000 C CNN
+F 1 "SW_DIP_x01" H 1700 8276 50  0000 C CNN
+F 2 "" H 1700 8100 50  0001 C CNN
+F 3 "~" H 1700 8100 50  0001 C CNN
+	1    1700 8100
+	1    0    0    -1
+$EndComp
+Text GLabel 1400 8100 0    50   Input ~ 0
+Switch
+$Comp
+L power:+BATT #PWR?
+U 1 1 5F51E639
+P 2000 8100
+F 0 "#PWR?" H 2000 7950 50  0001 C CNN
+F 1 "+BATT" H 2015 8273 50  0000 C CNN
+F 2 "" H 2000 8100 50  0001 C CNN
+F 3 "" H 2000 8100 50  0001 C CNN
+	1    2000 8100
+	0    1    1    0
+$EndComp
+$Comp
+L Device:R R?
+U 1 1 5F54C516
+P 14950 5050
+F 0 "R?" H 15150 5150 50  0000 R CNN
+F 1 "10k" H 15150 5050 50  0000 R CNN
+F 2 "Resistor_SMD:R_0805_2012Metric" V 14880 5050 50  0001 C CNN
+F 3 "~" H 14950 5050 50  0001 C CNN
+F 4 "C17414" H 14950 5050 50  0001 C CNN "LCSC"
+	1    14950 5050
+	1    0    0    -1
+$EndComp
+Wire Wire Line
+	14850 4850 14950 4850
+Wire Wire Line
+	14950 4900 14950 4850
+Connection ~ 14950 4850
+Wire Wire Line
+	14950 4850 15050 4850
+$Comp
+L power:GND #PWR?
+U 1 1 5F67F057
+P 14950 5200
+F 0 "#PWR?" H 14950 4950 50  0001 C CNN
+F 1 "GND" H 14955 5027 50  0000 C CNN
+F 2 "" H 14950 5200 50  0001 C CNN
+F 3 "" H 14950 5200 50  0001 C CNN
+	1    14950 5200
+	1    0    0    -1
 $EndComp
 $EndSCHEMATC

Commit message: Added switch and mosfet
Parts:
- added Q6: SiSS27DN, Package_SO:Vishay_PowerPAK_1212-8_Single, symbol Transistor_FET:SiSS27DN
- gave numbers to parts that had none: 2
Connections:
- net +BATT: now also R64.1; no longer SW1.2
- net GND: now also SW1.2; no longer R64.2
- net SRP: now also Q6.5 (D)
- net VCC: now also Q6.1 (S), Q6.2 (S), Q6.3 (S)
- net Switch: no longer names the net of SW1.1
- net Switch: now also R64.2, Q6.4 (G); no longer R64.1
Other:
- moved on the sheet: R64, SW1
Changed lines of the file:
@@
 	1    0    0    -1
 $EndComp
-$Comp
-L power:+BATT #PWR06
-U 1 1 5F077699
-P 9100 1100
-F 0 "#PWR06" H 9100 950 50  0001 C CNN
-F 1 "+BATT" H 9115 1273 50  0000 C CNN
-F 2 "" H 9100 1100 50  0001 C CNN
-F 3 "" H 9100 1100 50  0001 C CNN
-	1    9100 1100
-	1    0    0    -1
-$EndComp
 Wire Wire Line
 	8950 1150 9100 1150
@@
 Wire Wire Line
 	14550 4650 14550 4350
-Text GLabel 15050 4850 2    50   Input ~ 0
-Switch
 $Comp
-L Switch:SW_DIP_x01 SW?
+L Switch:SW_DIP_x01 SW1
 U 1 1 5F46B8F6
-P 1700 8100
-F 0 "SW?" H 1700 8367 50  0000 C CNN
-F 1 "SW_DIP_x01" H 1700 8276 50  0000 C CNN
-F 2 "" H 1700 8100 50  0001 C CNN
-F 3 "~" H 1700 8100 50  0001 C CNN
-	1    1700 8100
-	1    0    0    -1
-$EndComp
-Text GLabel 1400 8100 0    50   Input ~ 0
-Switch
-$Comp
-L power:+BATT #PWR?
-U 1 1 5F51E639
-P 2000 8100
-F 0 "#PWR?" H 2000 7950 50  0001 C CNN
-F 1 "+BATT" H 2015 8273 50  0000 C CNN
-F 2 "" H 2000 8100 50  0001 C CNN
-F 3 "" H 2000 8100 50  0001 C CNN
-	1    2000 8100
-	0    1    1    0
+P 15350 4850
+F 0 "SW1" H 15350 5000 50  0000 C CNN
+F 1 "SW_DIP_x01" H 15350 4700 50  0000 C CNN
+F 2 "" H 15350 4850 50  0001 C CNN
+F 3 "~" H 15350 4850 50  0001 C CNN
+	1    15350 4850
+	1    0    0    -1
 $EndComp
 $Comp
-L Device:R R?
+L Device:R R64
 U 1 1 5F54C516
-P 14950 5050
-F 0 "R?" H 15150 5150 50  0000 R CNN
-F 1 "10k" H 15150 5050 50  0000 R CNN
-F 2 "Resistor_SMD:R_0805_2012Metric" V 14880 5050 50  0001 C CNN
-F 3 "~" H 14950 5050 50  0001 C CNN
-F 4 "C17414" H 14950 5050 50  0001 C CNN "LCSC"
-	1    14950 5050
+P 14950 4700
+F 0 "R64" H 15150 4800 50  0000 R CNN
+F 1 "10k" H 15150 4700 50  0000 R CNN
+F 2 "Resistor_SMD:R_0805_2012Metric" V 14880 4700 50  0001 C CNN
+F 3 "~" H 14950 4700 50  0001 C CNN
+F 4 "C17414" H 14950 4700 50  0001 C CNN "LCSC"
+	1    14950 4700
 	1    0    0    -1
 $EndComp
 Wire Wire Line
 	14850 4850 14950 4850
-Wire Wire Line
-	14950 4900 14950 4850
 Connection ~ 14950 4850
 Wire Wire Line
 	14950 4850 15050 4850
 $Comp
-L power:GND #PWR?
-U 1 1 5F67F057
-P 14950 5200
-F 0 "#PWR?" H 14950 4950 50  0001 C CNN
-F 1 "GND" H 14955 5027 50  0000 C CNN
-F 2 "" H 14950 5200 50  0001 C CNN
-F 3 "" H 14950 5200 50  0001 C CNN
-	1    14950 5200
+L Transistor_FET:SiSS27DN Q6
+U 1 1 5F2D0B49
+P 14650 4850
+F 0 "Q6" H 14855 4804 50  0000 L CNN
+F 1 "SiSS27DN" H 14855 4895 50  0000 L CNN
+F 2 "Package_SO:Vishay_PowerPAK_1212-8_Single" H 14850 4775 50  0001 L CIN
+F 3 "http://www.vishay.com/docs/62847/siss27dn.pdf" V 14650 4850 50  0001 L CNN
+	1    14650 4850
+	-1   0    0    1
+$EndComp
+$Comp
+L power:+BATT #PWR06
+U 1 1 5F077699
+P 9100 1100
+F 0 "#PWR06" H 9100 950 50  0001 C CNN
+F 1 "+BATT" H 9115 1273 50  0000 C CNN
+F 2 "" H 9100 1100 50  0001 C CNN
+F 3 "" H 9100 1100 50  0001 C CNN
+	1    9100 1100
+	1    0    0    -1
+$EndComp
+$Comp
+L power:+BATT #PWR0120
+U 1 1 5F3B58EA
+P 14950 4550
+F 0 "#PWR0120" H 14950 4400 50  0001 C CNN
+F 1 "+BATT" H 14965 4723 50  0000 C CNN
+F 2 "" H 14950 4550 50  0001 C CNN
+F 3 "" H 14950 4550 50  0001 C CNN
+	1    14950 4550
 	1    0    0    -1
 $EndComp
+$Comp
+L power:GND #PWR0121
+U 1 1 5F3C4D8C
+P 15650 4850
+F 0 "#PWR0121" H 15650 4600 50  0001 C CNN
+F 1 "GND" H 15655 4677 50  0000 C CNN
+F 2 "" H 15650 4850 50  0001 C CNN
+F 3 "" H 15650 4850 50  0001 C CNN
+	1    15650 4850
+	0    -1   -1   0
+$EndComp
 $EndSCHEMATC

Commit message: started organizing layout
Parts:
- J7: footprint Connector_JST:JST_PH_B5B-PH-K_1x05_P2.00mm_Vertical -> Connector_JST:JST_PH_B2B-PH-K_1x02_P2.00mm_Vertical
- SW1: footprint (none) -> SS-12D28L4:SS-12D28L4; symbol Switch:SW_DIP_x01 -> Switch:SW_SPDT
Connections:
- net GND: now also SW1.1 (A); no longer SW1.2
- net at Q6.4 (G), R64.2: now also SW1.2 (B); no longer SW1.1
Changed lines of the file:
@@
 F 0 "J7" H 5500 5800 50  0000 C CNN
 F 1 "Side_Brush" H 5650 5700 50  0000 C CNN
-F 2 "Connector_JST:JST_PH_B5B-PH-K_1x05_P2.00mm_Vertical" H 5350 5800 50  0001 C CNN
+F 2 "Connector_JST:JST_PH_B2B-PH-K_1x02_P2.00mm_Vertical" H 5350 5800 50  0001 C CNN
 F 3 "~" H 5350 5800 50  0001 C CNN
 	1    5350 5800
@@
 	14550 4650 14550 4350
 $Comp
-L Switch:SW_DIP_x01 SW1
+L Switch:SW_SPDT SW1
 U 1 1 5F46B8F6
-P 15350 4850
-F 0 "SW1" H 15350 5000 50  0000 C CNN
-F 1 "SW_DIP_x01" H 15350 4700 50  0000 C CNN
-F 2 "" H 15350 4850 50  0001 C CNN
-F 3 "~" H 15350 4850 50  0001 C CNN
-	1    15350 4850
+P 15250 4850
+F 0 "SW1" H 15250 5000 50  0000 C CNN
+F 1 "SW_DIP_x01" H 15250 4700 50  0000 C CNN
+F 2 "SS-12D28L4:SS-12D28L4" H 15250 4850 50  0001 C CNN
+F 3 "~" H 15250 4850 50  0001 C CNN
+	1    15250 4850
 	1    0    0    -1
 $EndComp
@@
 L power:GND #PWR0121
 U 1 1 5F3C4D8C
-P 15650 4850
-F 0 "#PWR0121" H 15650 4600 50  0001 C CNN
-F 1 "GND" H 15655 4677 50  0000 C CNN
-F 2 "" H 15650 4850 50  0001 C CNN
-F 3 "" H 15650 4850 50  0001 C CNN
-	1    15650 4850
+P 15450 4750
+F 0 "#PWR0121" H 15450 4500 50  0001 C CNN
+F 1 "GND" H 15455 4577 50  0000 C CNN
+F 2 "" H 15450 4750 50  0001 C CNN
+F 3 "" H 15450 4750 50  0001 C CNN
+	1    15450 4750
 	0    -1   -1   0
 $EndComp

Commit message: working on the layout, fixes on the schematic
Parts:
- added F?: Fuse, symbol Device:Fuse
- J10: footprint Connector_JST:JST_PH_B4B-PH-K_1x04_P2.00mm_Vertical -> Connector_JST:JST_PH_S4B-PH-K_1x04_P2.00mm_Horizontal
Connections:
- net +BATT: now also F?.1; no longer J1.2 (Pin_2)
- new net: F?.2, J1.2 (Pin_2)
Other:
- moved on the sheet: J1
Changed lines of the file:
@@
 L Connector_Generic:Conn_01x02 J1
 U 1 1 5F03E4EC
-P 8750 1250
-F 0 "J1" H 8900 1250 50  0000 C CNN
-F 1 "Main_Batt_Con" H 8950 1350 50  0000 C CNN
-F 2 "Connector_AMASS:AMASS_XT30UPB-M_1x02_P5.0mm_Vertical" H 8750 1250 50  0001 C CNN
-F 3 "~" H 8750 1250 50  0001 C CNN
-F 4 "C428721" H 8750 1250 50  0001 C CNN "LCSC"
-	1    8750 1250
+P 8450 1250
+F 0 "J1" H 8600 1250 50  0000 C CNN
+F 1 "Main_Batt_Con" H 8650 1350 50  0000 C CNN
+F 2 "Connector_AMASS:AMASS_XT30UPB-M_1x02_P5.0mm_Vertical" H 8450 1250 50  0001 C CNN
+F 3 "~" H 8450 1250 50  0001 C CNN
+F 4 "C428721" H 8450 1250 50  0001 C CNN "LCSC"
+	1    8450 1250
 	-1   0    0    1
 $EndComp
@@
 	8950 1150 9100 1150
 Wire Wire Line
-	8950 1250 9100 1250
-Wire Wire Line
 	9100 1250 9100 1800
 Wire Wire Line
@@
 F 0 "J10" H 8030 10392 50  0000 L CNN
 F 1 "SWD" H 8030 10301 50  0000 L CNN
-F 2 "Connector_JST:JST_PH_B4B-PH-K_1x04_P2.00mm_Vertical" H 7950 10350 50  0001 C CNN
+F 2 "Connector_JST:JST_PH_S4B-PH-K_1x04_P2.00mm_Horizontal" H 7950 10350 50  0001 C CNN
 F 3 "~" H 7950 10350 50  0001 C CNN
 	1    7950 10350
@@
 	0    -1   -1   0
 $EndComp
+$Comp
+L Device:Fuse F?
+U 1 1 5F46259D
+P 8800 1150
+F 0 "F?" V 8603 1150 50  0000 C CNN
+F 1 "Fuse" V 8694 1150 50  0000 C CNN
+F 2 "" V 8730 1150 50  0001 C CNN
+F 3 "~" H 8800 1150 50  0001 C CNN
+	1    8800 1150
+	0    1    1    0
+$EndComp
+Wire Wire Line
+	8650 1250 9100 1250
 $EndSCHEMATC

Commit message: more layout stuff
Parts:
- removed F?: Fuse, symbol Device:Fuse
- added F1: Polyfuse, 16R1400GH:16R1400GH, symbol Device:Polyfuse
- added F?: Fuse, symbol Device:Fuse
Connections:
- net +5V: now also J11.3 (Pin_3); no longer J11.1 (Pin_1)
- net +BATT: now also F?.1
- net GND: now also J11.1 (Pin_1), J11.2 (Pin_2); no longer J11.3 (Pin_3), J11.4 (Pin_4)
- net VCC: now also J11.4 (Pin_4); no longer J11.2 (Pin_2)
- net at J1.2 (Pin_2): now also F1.2
- new net: F1.1, F?.2
Other:
- moved on the sheet: J1
Changed lines of the file:
@@
 L Connector_Generic:Conn_01x02 J1
 U 1 1 5F03E4EC
-P 8450 1250
-F 0 "J1" H 8600 1250 50  0000 C CNN
-F 1 "Main_Batt_Con" H 8650 1350 50  0000 C CNN
-F 2 "Connector_AMASS:AMASS_XT30UPB-M_1x02_P5.0mm_Vertical" H 8450 1250 50  0001 C CNN
-F 3 "~" H 8450 1250 50  0001 C CNN
-F 4 "C428721" H 8450 1250 50  0001 C CNN "LCSC"
-	1    8450 1250
+P 8150 1250
+F 0 "J1" H 8300 1250 50  0000 C CNN
+F 1 "Main_Batt_Con" H 8350 1350 50  0000 C CNN
+F 2 "Connector_AMASS:AMASS_XT30UPB-M_1x02_P5.0mm_Vertical" H 8150 1250 50  0001 C CNN
+F 3 "~" H 8150 1250 50  0001 C CNN
+F 4 "C428721" H 8150 1250 50  0001 C CNN "LCSC"
+	1    8150 1250
 	-1   0    0    1
 $EndComp
@@
 L power:+5V #PWR0117
 U 1 1 5F4EF8D3
-P 3250 7900
-F 0 "#PWR0117" H 3250 7750 50  0001 C CNN
-F 1 "+5V" H 3265 8073 50  0000 C CNN
-F 2 "" H 3250 7900 50  0001 C CNN
-F 3 "" H 3250 7900 50  0001 C CNN
-	1    3250 7900
-	1    0    0    -1
+P 3150 8200
+F 0 "#PWR0117" H 3150 8050 50  0001 C CNN
+F 1 "+5V" V 3150 8400 50  0000 C CNN
+F 2 "" H 3150 8200 50  0001 C CNN
+F 3 "" H 3150 8200 50  0001 C CNN
+	1    3150 8200
+	0    -1   -1   0
 $EndComp
 $Comp
 L power:VCC #PWR0118
 U 1 1 5F4F5FDB
-P 3100 7900
-F 0 "#PWR0118" H 3100 7750 50  0001 C CNN
-F 1 "VCC" H 3115 8073 50  0000 C CNN
-F 2 "" H 3100 7900 50  0001 C CNN
-F 3 "" H 3100 7900 50  0001 C CNN
-	1    3100 7900
-	1    0    0    -1
+P 3150 8300
+F 0 "#PWR0118" H 3150 8150 50  0001 C CNN
+F 1 "VCC" V 3150 8500 50  0000 C CNN
+F 2 "" H 3150 8300 50  0001 C CNN
+F 3 "" H 3150 8300 50  0001 C CNN
+	1    3150 8300
+	0    -1   -1   0
 $EndComp
 $Comp
 L power:GND #PWR0119
 U 1 1 5F4F9ED2
-P 3250 8400
-F 0 "#PWR0119" H 3250 8150 50  0001 C CNN
-F 1 "GND" H 3255 8227 50  0000 C CNN
-F 2 "" H 3250 8400 50  0001 C CNN
-F 3 "" H 3250 8400 50  0001 C CNN
-	1    3250 8400
-	1    0    0    -1
+P 3150 8050
+F 0 "#PWR0119" H 3150 7800 50  0001 C CNN
+F 1 "GND" V 3150 7850 50  0000 C CNN
+F 2 "" H 3150 8050 50  0001 C CNN
+F 3 "" H 3150 8050 50  0001 C CNN
+	1    3150 8050
+	0    1    1    0
 $EndComp
 Wire Wire Line
-	3350 8000 3250 8000
-Wire Wire Line
-	3250 8000 3250 7900
-Wire Wire Line
-	3100 7900 3100 8100
-Wire Wire Line
-	3100 8100 3350 8100
-Wire Wire Line
-	3350 8200 3250 8200
-Wire Wire Line
-	3250 8200 3250 8300
-Wire Wire Line
-	3350 8300 3250 8300
-Connection ~ 3250 8300
-Wire Wire Line
-	3250 8300 3250 8400
-Wire Wire Line
 	7000 10350 7750 10350
 Wire Wire Line
@@
 $EndComp
 $Comp
+L Device:Polyfuse F1
+U 1 1 5F382FA0
+P 8500 1150
+F 0 "F1" V 8275 1150 50  0000 C CNN
+F 1 "Polyfuse" V 8366 1150 50  0000 C CNN
+F 2 "16R1400GH:16R1400GH" H 8550 950 50  0001 L CNN
+F 3 "~" H 8500 1150 50  0001 C CNN
+	1    8500 1150
+	0    1    1    0
+$EndComp
+Wire Wire Line
+	3350 8000 3250 8000
+Wire Wire Line
+	3250 8000 3250 8050
+Wire Wire Line
+	3250 8050 3150 8050
+Wire Wire Line
+	3250 8050 3250 8100
+Wire Wire Line
+	3250 8100 3350 8100
+Connection ~ 3250 8050
+Wire Wire Line
+	3150 8200 3350 8200
+Wire Wire Line
+	3150 8300 3350 8300
+$Comp
 L Device:Fuse F?
-U 1 1 5F46259D
+U 1 1 5F7D6D82
 P 8800 1150
 F 0 "F?" V 8603 1150 50  0000 C CNN
@@
 $EndComp
 Wire Wire Line
-	8650 1250 9100 1250
+	8350 1250 9100 1250
 $EndSCHEMATC
