File: motorcon/motorcon.kicad_pcb (KiCad board)
At the start: 2 copper layers, 143 parts, among them J1 Main_Batt_Con, J10 SWD, J2 Batt_Balancer_Con, J3 Charger_Con, J4 Left_Motor, J5 Right_Motor, J6 Brush_Motor, J7 Side_Brush, J8 Conn_01x06, J9 SPI_PI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

Commit message: started pcb work
Parts:
- added J11: Main_Power, Connector_Molex:Molex_Mini-Fit_Jr_5569-04A2_2x02_P4.20mm_Horizontal, F.Cu at (-103.5, 124.9)
- C40, C42: footprint Capacitor_SMD:C_Elec_10x10.2 -> Capacitor_SMD:CP_Elec_10x10
- D3: footprint Diode_SMD:D_SOT-23_ANK -> Diode_SMD:D_SMB
- J3: footprint Connector_AMASS:AMASS_XT30PW-M_1x02_P2.50mm_Horizontal -> Connector_JST:JST_VH_B2P-VH_1x02_P3.96mm_Vertical
- L2: value 10H -> 10uH
- Q2: footprint Resistor_SMD:R_0805_2012Metric -> CSD87312Q3E:CSD87312Q3E
- Q3: footprint Resistor_SMD:R_0805_2012Metric -> CSD25402Q3A:CSD25402Q3A
- Q4, Q5: footprint Resistor_SMD:R_0805_2012Metric -> CSD17307Q5A:CSD17307Q5A
- R24, R28: footprint Resistor_SMD:R_0805_2012Metric -> Resistor_SMD:R_1206_3216Metric
- moved U1 128.4 mm to (-73.1, 161.3)
- moved R4 126.5 mm to (-52.0, 168.5)
- moved D2 125.9 mm to (-69.7, 169.2)
- moved R27 121.7 mm to (-47.6, 166.6)
- moved R3 119.8 mm to (-40.0, 157.8)
- moved Q5 117.1 mm to (-87.1, 167.9)
- moved C17 117.1 mm to (-44.4, 154.8)
- moved Y1 113.2 mm to (-74.5, 169.2)
- moved R14 111.0 mm to (-40.0, 154.8)
- moved Q1 109.7 mm to (-45.1, 147.4)
- moved R26 109.1 mm to (-39.7, 160.7)
- moved R32 109.1 mm to (-44.1, 163.7)
- moved U8 108.7 mm to (-65.9, 149.6)
- moved R44 104.4 mm to (-43.1, 169.6)
- moved R5 103.1 mm to (-31.0, 147.1)
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Connections:
- R55 pad 1: Net-(D4-Pad1) -> +3V3
- R55 pad 2: GND -> Net-(D4-Pad1)
