File: motorcon/motorcon.kicad_pcb (KiCad board)
At the start: 2 copper layers, 144 parts, among them J1 Main_Batt_Con, J10 SWD, J11 Main_Power, J2 Batt_Balancer_Con, J3 Charger_Con, J4 Left_Motor, J5 Right_Motor, J6 Brush_Motor, J7 Side_Brush, J8 Conn_01x06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

Commit message: started organizing layout
Parts:
- added Q6: SiSS27DN, Package_SO:Vishay_PowerPAK_1212-8_Single, F.Cu at (120.5, 79.9)
- added R63: 1M, Resistor_SMD:R_0805_2012Metric, F.Cu at (108.2, 112.9)
- added R64: 10k, Resistor_SMD:R_0805_2012Metric, F.Cu at (125.4, 80.0)
- added SW1: SW_DIP_x01, SS-12D28L4:SS-12D28L4, F.Cu at (125.5, 66.0)
- J1: footprint Connector_AMASS:AMASS_XT30PW-M_1x02_P2.50mm_Horizontal -> Connector_AMASS:AMASS_XT30UPB-M_1x02_P5.0mm_Vertical
- J10: footprint Connector_PinHeader_2.54mm:PinHeader_1x03_P2.54mm_Horizontal -> Connector_JST:JST_PH_B4B-PH-K_1x04_P2.00mm_Vertical
- J2: footprint Connector_JST:JST_PH_S4B-PH-K_1x04_P2.00mm_Horizontal -> Connector_JST:JST_PH_B4B-PH-K_1x04_P2.00mm_Vertical
- J4, J5, J6: footprint Connector_JST:JST_PH_S5B-PH-SM4-TB_1x05-1MP_P2.00mm_Horizontal -> Connector_JST:JST_PH_B5B-PH-K_1x05_P2.00mm_Vertical
- J7: footprint Connector_JST:JST_PH_S2B-PH-SM4-TB_1x02-1MP_P2.00mm_Horizontal -> Connector_JST:JST_PH_B2B-PH-K_1x02_P2.00mm_Vertical
- J8: footprint Connector_JST:JST_PH_S6B-PH-SM4-TB_1x06-1MP_P2.00mm_Horizontal -> Connector_JST:JST_PH_B5B-PH-K_1x05_P2.00mm_Vertical
- J9: footprint Connector_JST:JST_PH_S4B-PH-SM4-TB_1x04-1MP_P2.00mm_Horizontal -> Connector_JST:JST_PH_B5B-PH-K_1x05_P2.00mm_Vertical
- moved J6 327.0 mm to (247.0, 98.3), turned to 90 degrees
- moved J4 316.6 mm to (246.9, 133.6), turned to 90 degrees
- moved U8 304.8 mm to (233.8, 94.2)
- moved R44 303.9 mm to (258.3, 130.6)
- moved R47 302.9 mm to (259.5, 91.1)
- moved R40 301.6 mm to (254.6, 96.5)
- moved C30 300.0 mm to (233.1, 90.4)
- moved J5 299.6 mm to (210.7, 156.8), turned to 90 degrees
- moved R48 296.5 mm to (259.3, 96.1)
- moved R32 291.8 mm to (238.3, 90.6)
- moved C35 289.4 mm to (209.7, 65.8)
- moved R36 286.6 mm to (253.2, 130.4)
- moved R43 286.5 mm to (258.5, 126.1)
- moved U7 283.8 mm to (197.6, 152.8)
- moved C39 282.9 mm to (221.9, 75.8)
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Connections:
- C24 pad 1: SRP -> VCC
- C25 pad 1: SRP -> VCC
- C26 pad 1: SRP -> VCC
- C27 pad 1: SRP -> VCC
- C28 pad 1: SRP -> VCC
- C29 pad 1: SRP -> VCC
- C30 pad 1: SRP -> VCC
- C31 pad 1: SRP -> VCC
- C32 pad 2: SRP -> VCC
- C33 pad 2: SRP -> VCC
- C34 pad 2: SRP -> VCC
- C35 pad 2: SRP -> VCC
- C40 pad 1: SRP -> VCC
- J10 pad 1: Net-(J10-Pad1) -> +3V3
- J10 pad 3: GND -> Net-(J10-Pad3)
- J11 pad 2: SRP -> VCC
- J4 pad 4: SRP -> VCC
- J5 pad 4: SRP -> VCC
- J6 pad 4: SRP -> VCC
- R35 pad 2: SRP -> VCC
- R37 pad 2: SRP -> VCC
- R39 pad 2: SRP -> VCC
- R41 pad 2: SRP -> VCC
- R43 pad 2: SRP -> VCC
- R45 pad 2: SRP -> VCC
- R47 pad 2: SRP -> VCC
- R49 pad 2: SRP -> VCC
- U1 pad 34: Net-(J10-Pad1) -> Net-(J10-Pad2)
- U1 pad 37: Net-(J10-Pad2) -> Net-(J10-Pad3)
- U5 pad 7: SRP -> VCC
- U6 pad 11: SRP -> VCC
- U7 pad 11: SRP -> VCC
- U8 pad 11: SRP -> VCC
- U9 pad 11: SRP -> VCC

Commit message: working on the layout, fixes on the schematic
Parts:
- J10: footprint Connector_JST:JST_PH_B4B-PH-K_1x04_P2.00mm_Vertical -> Connector_JST:JST_PH_S4B-PH-K_1x04_P2.00mm_Horizontal
- moved C39 103.2 mm to (160.9, 159.0)
- moved R50 103.2 mm to (170.4, 148.4)
- moved C31 103.2 mm to (153.7, 147.8)
- moved R30 103.2 mm to (148.4, 158.1)
- moved R34 103.2 mm to (153.6, 158.4)
- moved R41 103.2 mm to (166.6, 143.0)
- moved R42 103.2 mm to (171.5, 156.6)
- moved R49 103.2 mm to (171.0, 153.2)
- moved C35 101.6 mm to (145.2, 144.3)
- moved R28 101.2 mm to (149.5, 82.6), turned to 90 degrees
- moved J7 100.6 mm to (165.6, 153.0)
- moved U9 96.2 mm to (158.7, 151.2), turned to 90 degrees
- moved Q3 83.7 mm to (149.5, 77.5), turned to 270 degrees
- moved C27 76.0 mm to (159.6, 135.4), turned to 270 degrees
- moved J6 71.9 mm to (186.7, 137.3)
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Other:
- board outline added: 99.6 x 86.9 mm
- net class Batt added: clearance 0.2, trace_width 12.6, via_dia 0.8, via_drill 0.4

Commit message: more layout stuff
Parts:
- added F1: Polyfuse, 16R1400GH:16R1400GH, F.Cu at (141.4, 61.6)
- J1, J2, R64: moved to B.Cu
- moved R22 110.3 mm to (138.4, 114.2), turned to 180 degrees
- moved C8 106.4 mm to (138.4, 112.2)
- moved D2 106.0 mm to (151.0, 109.8)
- moved Q2 102.2 mm to (139.8, 109.0)
- moved U4 101.8 mm to (145.5, 114.2)
- moved Q5 100.0 mm to (142.0, 100.2), turned to 270 degrees
- moved R21 97.4 mm to (141.2, 114.3), turned to 90 degrees
- moved Q4 93.0 mm to (148.8, 100.2), turned to 90 degrees
- moved D1 83.2 mm to (132.5, 114.2)
- moved L1 82.4 mm to (144.6, 89.3), turned to 270 degrees
- moved J3 73.4 mm to (126.8, 101.2)
- moved C11 70.2 mm to (143.0, 110.8), turned to 90 degrees
- moved Q6 27.5 mm to (152.0, 87.2), turned to 90 degrees
- moved R64 24.7 mm to (127.2, 49.6), turned to 270 degrees
- moved C25 22.7 mm to (158.8, 122.2)
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Connections:
- J1 pad 2: +BATT -> Net-(F1-Pad2)
- J11 pad 1: +5V -> GND
- J11 pad 2: VCC -> GND
- J11 pad 3: GND -> +5V
- J11 pad 4: GND -> VCC
Routing:
- net Net-(F1-Pad2): track 0.00 -> 7.17 mm
